File: demoboard/demoboard.kicad_pcb (KiCad board)
At the start: 2 copper layers, 38.1 x 50.8 mm, 39 parts, among them CON1 BARREL_JACK, M1 ESP-07, P1 USB_OTG, P2 header1, Q1 BC547, Q2 BC547, SW1 UI1, SW2 UI1, U1 CH340G, U2 1117-5v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

Commit message: usb and esp 3d models
Parts:
- P1: footprint Connect:USB_Micro-B -> MolexMicroUSB:molex-microUSB
- moved P1 1.42 mm to (145.0, 122.2), turned to 0 degrees
Routing:
- net GND: track 110.0 -> 102.3 mm
- net VUSB: track 45.1 -> 46.1 mm
- net UD-: track 12.0 -> 11.4 mm
