File: demoboard/demoboard.sch (KiCad schematic (older format))
At the start: 14 parts, among them CON1 BARREL_JACK, P1 USB_OTG, U1 CH340G, U2 7805, U3 AP1117, Y1 Crystal

Commit message: added ESP
Parts:
- added M1: ESP-07, ESP-07:ESP-07, symbol ESP-07
- CON1: footprint (none) -> Connect:BARREL_JACK
- JP1, U2: footprint (none) -> Pin_Headers:Pin_Header_Straight_1x03
- Y1: footprint (none) -> Crystals:Crystal_HC50-U_Vertical
Connections:
- wire segments 50 -> 54

Commit message: layoutv1
Parts:
- removed C1: 100uf, symbol C
- removed C2: 10uf, symbol C_Small
- removed C3: 100uf, symbol C_Small
- removed C4: 1000uf, symbol C_Small
- removed U2: 7805, Pin_Headers:Pin_Header_Straight_1x03, symbol 7805
- added C10, C8: 0.1uf, Capacitors_SMD:C_1206_HandSoldering, symbol C_Small
- added C3, C4, C5, C6: 10uf, Capacitors_Tantalum_SMD:TantalC_SizeA_EIA-3216_HandSoldering, symbol CP_Small
- added C9: 1mf, Capacitors_Elko_ThroughHole:Elko_vert_11.2x6.3mm_RM2.5, symbol CP_Small
- added D1: GREEN, SMD_Packages:SMD-1206_Pol, symbol Led_Small
- added D2: RED, SMD_Packages:SMD-1206_Pol, symbol Led_Small
- added P2: header1, Pin_Headers:Pin_Header_Straight_1x05, symbol CONN_01X05
- added Q1, Q2: BC547, Housings_SOT-23_SOT-143_TSOT-6:SOT-23, symbol BC547
- added R1, R2, R3: 10K, Resistors_SMD:R_1206_HandSoldering, symbol R
- added R10, R9: 120E, Resistors_SMD:R_1206_HandSoldering, symbol R
- added R11: 100R, Resistors_SMD:R_1206_HandSoldering, symbol R
- added R4: 220R, Resistors_SMD:R_1206_HandSoldering, symbol R
- added R5, R6, R7: 1K, Resistors_SMD:R_1206_HandSoldering, symbol R
- added R8: 1.5K, Resistors_SMD:R_1206_HandSoldering, symbol R
- added RV1: 10K, Potentiometers:Potentiometer_Bourns_3296W_3-8Zoll_Inline_ScrewUp, symbol POT
- added SW1: PGM, Buttons_Switches_SMD:SW_SPST_FSMSM, symbol SW_PUSH
- added SW2, SW3: UI1, Buttons_Switches_SMD:SW_SPST_FSMSM, symbol SW_PUSH
- added U2: AP1117, TO_SOT_Packages_SMD:SOT-223, symbol AP1117
- added W1: ws2812b, WS2812b:ws2812B, symbol ws2812b
- C1: renamed from C5; footprint (none) -> Capacitors_SMD:C_1206_HandSoldering
- C2: renamed from C6; footprint (none) -> Capacitors_SMD:C_1206_HandSoldering
- C7: value C_Small -> 0.1uf; footprint (none) -> Capacitors_SMD:C_1206_HandSoldering
- P1: footprint (none) -> Connect:USB_Micro-B
- U3: footprint (none) -> TO_SOT_Packages_SMD:SOT-223
- Y1: value Crystal -> 12MHz
Connections:
- net +3V3: now also M1.14 (CH_PD), C6.1, C8.1, P2.4 (P4), R2.2, R3.2, R4.1
- net +5V: now also C10.1, C5.1, P2.3 (P3), R6.2, R8.2, W1.1 (VDD)
- net 12v: now also C3.1, C9.1, U2.3 (VI)
- net GND: now also C10.2, C3.2, C4.2, C5.2, C6.2, C8.2, C9.2, D1.1 (K), D2.1 (K), P2.5 (P5), Q1.3 (E), Q2.3 (E), R1.2, R11.2, RV1.3, SW1.1, SW2.2, SW3.2, U2.1 (GND/ADJ), W1.3 (VSS)
- net RX: now also M1.1 (TXD); no longer M1.2 (RXD)
- net TX: now also M1.2 (RXD); no longer M1.1 (TXD)
- net UD+: now also P1.3 (D+)
- net UD-: now also P1.2 (D-)
- net at M1.10 (GPIO13): now also R9.1
- net at M1.11 (GPIO12): now also R10.1
- net at M1.12 (GPIO14): now also R3.1, SW3.1
- net at M1.13 (GPIO16): now also R2.1, SW2.1
- net at M1.15 (ADC): now also RV1.2
- net JP1.1: now reaches M1.3 (GPIO4)
- net JP1.1: now also P2.1 (P1)
- net JP1.2: now reaches M1.4 (GPIO5)
- net JP1.2: now also P2.2 (P2)
- net at M1.5 (GPIO0): now also SW1.2
- net 3v3In: now reaches M1.6 (GPIO2)
- net 3v3In: now also R5.2
- net at M1.7 (GPIO15): now also R1.1
- net VLDO renamed VLDO5v
- net VLDO5v: now also C4.1, U2.2 (VO)
- new net: Q2.2 (B), R7.1
- new net: Q1.1 (C), R6.1, R7.2
- new net: Q1.2 (B), R5.1
- new net: R11.1, R4.2, RV1.1
- new net: D2.2 (A), R10.2
- new net: D1.2 (A), R9.2
- new net 5vOut: Q2.1 (C), R8.1, W1.4 (DIn)
- no-connect marks 6 -> 9
Other:
- note added: "3v3 - 5v Tx"
- moved on the sheet: C1, C2, CON1, JP1, P1, U1, U3, Y1

Commit message: usb and esp 3d models
Parts:
- P1: footprint Connect:USB_Micro-B -> MolexMicroUSB:molex microUSB
Changed lines of the file:
@@
 F 0 "P1" H 10575 3875 50  0000 C CNN
 F 1 "USB_OTG" H 10250 4200 50  0000 C CNN
-F 2 "Connect:USB_Micro-B" V 10200 3900 60  0001 C CNN
-F 3 "" V 10200 3900 60  0000 C CNN
+F 2 "MolexMicroUSB:molex microUSB" V 10200 3900 60  0001 C CNN
+F 3 "http://www.molex.com/pdm_docs/sd/473460001_sd.pdf" V 10200 3900 60  0001 C CNN
 	1    10250 4000
 	0    1    1    0
